File: InputASRC_RS485.sch (KiCad schematic (older format))
At the start: 0 parts

Commit message: HDMI input board
Parts:
- added R? (x2): RES, symbol RES
Changed lines of the file:
@@
 LIBS:contrib
 LIBS:valves
+LIBS:InputASRC-cache
 EELAYER 27 0
 EELAYER END
 $Descr A4 11693 8268
 encoding utf-8
-Sheet 1 5
+Sheet 2 6
 Title ""
 Date "9 aug 2013"
@@
 Comment4 ""
 $EndDescr
+$Comp
+L RES R?
+U 1 1 52053430
+P 6850 2400
+F 0 "R?" H 6510 2450 60  0000 C CNN
+F 1 "RES" H 7150 2450 60  0000 C CNN
+F 2 "" H 6850 2400 60  0000 C CNN
+F 3 "" H 6850 2400 60  0000 C CNN
+	1    6850 2400
+	1    0    0    -1
+$EndComp
+$Comp
+L RES R?
+U 1 1 5205344E
+P 6850 2600
+F 0 "R?" H 6510 2650 60  0000 C CNN
+F 1 "RES" H 7150 2650 60  0000 C CNN
+F 2 "" H 6850 2600 60  0000 C CNN
+F 3 "" H 6850 2600 60  0000 C CNN
+	1    6850 2600
+	1    0    0    -1
+$EndComp
 $EndSCHEMATC
